File: Encoder_board.kicad_sch (KiCad schematic)
At the start: 16 parts, among them U1 XT60_M, U2 BP5293-50, U3 BA033CC0FP

Commit message: 回路図を書き進めた（未完）
Parts:
- added C10, C11, C12, C13, C15, C8, C9: 0.1u, Capacitor_SMD:C_0603_1608Metric_Pad1.08x0.95mm_HandSolder, symbol Device:C
- added C14, C16: 0.1u, symbol Device:C
- added D6, D7, D8, D9: LED, symbol Device:LED
- added J1, J2, J3, J4, J6: Conn_01x05_Socket_Encoder1, symbol Connector:Conn_01x05_Socket
- added J5: RS485, Connector_PinHeader_2.54mm:PinHeader_1x04_P2.54mm_Vertical, symbol Connector:Conn_01x04_Socket
- added R1, R10, R11, R12, R13, R2, R6, R7, R8, R9: 4.7k, symbol Device:R
- added R14, R16, R17, R19: 2.2k, Resistor_SMD:R_0603_1608Metric_Pad0.98x0.95mm_HandSolder, symbol Device:R
- added R15, R18: 120, Resistor_SMD:R_0603_1608Metric_Pad0.98x0.95mm_HandSolder, symbol Device:R
- added R20, R4, R5: 1k, symbol Device:R
- added R3: 10k, symbol Device:R
- added SW1: SW_Reset, symbol Switch:SW_Push
- added SW2: SW_DIP_x02_CANnum, symbol Switch:SW_DIP_x02
- added U4: TXRX_pokayoke, MyLib:TXRX_pokayoke, symbol txrx_pokayoke:TXRX_pokayoke
- added U5: STM32G431KBTx, Package_QFP:LQFP-32_7x7mm_P0.8mm, symbol MCU_ST_STM32G4:STM32G431KBTx
- added U6, U7: UTRS485G-S08-R, Package_SO:SOP-8_3.9x4.9mm_P1.27mm, symbol Interface_UART:MAX3485
Connections:
- net +12V: now also R3.1
- net +3.3V: now also C14.1, R5.1, SW2.1, SW2.2, U5.1 (VDD), U5.12 (PA7), U5.13 (PB0)
- net +5V: now also C10.1, C11.1, C12.1, C13.1, C15.1, C8.1, C9.1, J1.4 (Pin_4), J2.4 (Pin_4), J3.4 (Pin_4), J4.4 (Pin_4), J6.4 (Pin_4), R14.2, R17.2, R4.1, U6.2 (~{RE}), U6.3 (DE), U6.8 (VCC), U7.8 (VCC)
- net GND: now also C10.2, C11.2, C12.2, C13.2, C14.2, C15.2, C16.1, C8.2, C9.2, D6.1 (K), D7.1 (K), D8.1 (K), D9.1 (K), J1.1 (Pin_1), J2.1 (Pin_1), J3.1 (Pin_1), J4.1 (Pin_1), J6.1 (Pin_1), R1.2, R10.2, R11.2, R12.2, R13.2, R16.1, R19.1, R2.2, R6.2, R7.2, R8.2, R9.2, SW1.1, SW2.3, SW2.4, U5.16 (VSS), U5.32 (VSS), U6.5 (GND), U7.2 (~{RE}), U7.3 (DE), U7.5 (GND)
- new net: C16.2, SW1.2, U5.4 (PG10)
- new net: U4.2 (RX2), U7.1 (RO)
- new net: U4.4 (TX2), U6.4 (DI)
- new net: D8.2 (A), R5.2
- new net: J5.1 (Pin_1), R15.1, R16.2, U6.6 (A)
- new net: D9.2 (A), R20.2
- new net: D7.2 (A), R4.2
- new net: J5.2 (Pin_2), R14.1, R15.2, U6.7 (B)
- new net: J5.3 (Pin_3), R18.1, R19.2, U7.6 (A)
- new net: D6.2 (A), R3.2
- new net: J5.4 (Pin_4), R17.1, R18.2, U7.7 (B)
- new net En1_A: J1.3 (Pin_3), J2.3 (Pin_3), J3.3 (Pin_3), J4.3 (Pin_3), J6.3 (Pin_3), R1.1, R10.1, R12.1, R6.1, R8.1
- new net En1_B: J1.5 (Pin_5), J2.5 (Pin_5), J3.5 (Pin_5), J4.5 (Pin_5), J6.5 (Pin_5), R11.1, R13.1, R2.1, R7.1, R9.1
- new net RS485_RX: U4.3 (RX1)
- new net RS485_TX: U4.1 (TX1)
- new net User_LED: R20.1, U5.10 (PA5)
- no-connect marks 0 -> 11
Other:
- note added: "5V"
- note added: "A"
- note added: "B"
- note added: "ENCODER"
- note added: "G431 KBT6"
- note added: "GND"
- note added: "LED"
- note added: "RS485"
- note added: "X"
- moved on the sheet: C1, C2, C3, C4, C5, C6, C7, D1, D2, D3, D4, D5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

Commit message: 回路図を一応完成。ミスがないか、動作するか確認する
Parts:
- added C1: 0.1u, symbol Device:C
- added C2: 0.1u, Capacitor_SMD:C_0603_1608Metric_Pad1.08x0.95mm_HandSolder, symbol Device:C
- added J2: CAN_OUT, symbol Connector:Conn_01x02_Socket
- added J7: Write_G431, symbol Connector:Conn_01x06_Pin
- added R22, R23, R24: 10k, symbol Device:R
- added R7: 120, Resistor_SMD:R_0603_1608Metric_Pad0.98x0.95mm_HandSolder, symbol Device:R
- added SW1: SW_Boot, symbol Switch:SW_Push
- added SW4: SW_User, symbol Switch:SW_Push
- added U5: MCP2562-E-P, Package_DIP:DIP-8_W7.62mm, symbol Interface_CAN_LIN:MCP2562-E-P
- renumbered C15 to C10, C5 to C11, C6 to C12, C7 to C13, C10 to C14, C13 to C15, C14 to C16, C16 to C17, C11 to C18, C8 to C3, C9 to C4, C2 to C5, C1 to C6, C4 to C7, C3 to C8, C12 to C9, D3 to D2, D2 to D3, D5 to D4, D6 to D5, D7 to D6, D4 to D7, J5 to J1, J6 to J4, J1 to J5, J4 to J6, J2 to J8, R18 to R1, R9 to R10, R13 to R11, R3 to R12, R4 to R13, R5 to R14, R1 to R15, R10 to R16, R2 to R17, R11 to R18, R6 to R19, R15 to R2, R7 to R20, R20 to R21, R14 to R3, R16 to R4, R17 to R5, R19 to R6, R12 to R9, SW1 to SW2, SW2 to SW3, U4 to U2, U6 to U3, U7 to U4, U2 to U6, U3 to U7, U5 to U8
Connections:
- net +3.3V: now also R22.1, R23.1, R24.1, SW1.1; no longer SW3.1, SW3.2, U8.12 (PA7), U8.13 (PB0)
- net +5V: now also C2.1, J7.1 (Pin_1), U5.3 (VDD)
- net En1_A: now also U8.18 (PA8)
- net En1_B: now also U8.19 (PA9)
- net En2_A: now also U8.5 (PA0)
- net En2_B: now also U8.6 (PA1)
- net En3_A: now also U8.11 (PA6)
- net En3_B: now also U8.9 (PA4)
- net En4_A: now also U8.29 (PB6)
- net En4_B: now also U8.30 (PB7)
- net En5_A: now also U8.25 (PA15)
- net En5_B: now also U8.31 (PB8), SW1.2
- net GND: now also C1.2, C2.2, J7.3 (Pin_3), SW4.2, U5.2 (VSS), U5.8 (STBY)
- net RS485_RX: now also U8.8 (PA3), J7.4 (Pin_4)
- net RS485_TX: now also U8.7 (PA2), J7.5 (Pin_5)
- net CAN_RD: now reaches U8.21 (PA11)
- net CAN_RD: now also U5.4 (RXD)
- net CAN_TD: now reaches U8.22 (PA12)
- net CAN_TD: now also U5.1 (TXD)
- net User_button: now reaches U8.28 (PB5)
- net User_button: now also R24.2, SW4.1
- new net: J2.1 (Pin_1), R7.1, U5.7 (CANH)
- new net: J2.2 (Pin_2), R7.2, U5.6 (CANL)
- new net +3V3: C1.1, U5.5 (Vio)
- new net CAN_num1: R22.2, SW3.1, U8.12 (PA7)
- new net CAN_num2: R23.2, SW3.2, U8.13 (PB0)
- no-connect marks 11 -> 19
Other:
- note added: "CAN"
- note removed: "LED"
- moved on the sheet: C10, C11, C12, C13, C14, C15, C16, C17, C18, C3, C4, C5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

Commit message: 少し修正
Connections:
- net En1_A: no longer J3.3 (Pin_3), J5.3 (Pin_3), J6.3 (Pin_3), J8.3 (Pin_3), R15.1, R16.1, R19.1, R8.1
- net En1_B: no longer J3.5 (Pin_5), J5.5 (Pin_5), J6.5 (Pin_5), J8.5 (Pin_5), R10.1, R17.1, R18.1, R20.1
- net En2_A: now also J5.3 (Pin_3), R15.1
- net En2_B: now also J5.5 (Pin_5), R17.1
- net En3_A: now also J8.3 (Pin_3), R19.1
- net En3_B: now also J8.5 (Pin_5), R20.1
- net En4_A: now also J3.3 (Pin_3), R8.1
- net En4_B: now also J3.5 (Pin_5), R10.1
- net En5_A: now also J6.3 (Pin_3), R16.1
- net En5_B: now also J6.5 (Pin_5), R18.1

Commit message: 回路図完成
Parts:
- removed C18: 0.1u, Capacitor_SMD:C_0603_1608Metric_Pad1.08x0.95mm_HandSolder, symbol Device:C
- removed D4, D7: 1N4148, MyLib:SOD123, symbol Device:D
- removed D5, D8: LED, symbol Device:LED
- removed J1: RS485, Connector_PinHeader_2.54mm:PinHeader_1x04_P2.54mm_Vertical, symbol Connector:Conn_01x04_Socket
- removed J7: Write_G431, symbol Connector:Conn_01x06_Pin
- removed U2: TXRX_pokayoke, MyLib:TXRX_pokayoke, symbol txrx_pokayoke:TXRX_pokayoke
- removed U4: UTRS485G-S08-R, Package_SO:SOP-8_3.9x4.9mm_P1.27mm, symbol Interface_UART:MAX3485
- removed U5: MCP2562-E-P, Package_DIP:DIP-8_W7.62mm, symbol Interface_CAN_LIN:MCP2562-E-P
- removed U7: BA033CC0FP, Package_TO_SOT_SMD:TO-252-2, symbol bp5293-50:L7805
- removed U8: STM32G431KBTx, Package_QFP:LQFP-32_7x7mm_P0.8mm, symbol MCU_ST_STM32G4:STM32G431KBTx
- added D4, D7: LED, LED_THT:LED_D3.0mm, symbol Device:LED
- added D5, D8: 1N4148, mylib:SOD123, symbol Device:D
- added J1: Conn_01x05_Socket_RS485, Connector_JST:JST_XH_B5B-XH-A_1x05_P2.50mm_Vertical, symbol Connector:Conn_01x05_Socket
- added J7: ST-Link_pinsocket, Connector_PinSocket_2.54mm:PinSocket_2x06_P2.54mm_Vertical, symbol Connector_Generic:Conn_02x06_Odd_Even
- added R24: 10k, Resistor_SMD:R_0603_1608Metric_Pad0.98x0.95mm_HandSolder, symbol Device:R
- added U2: UTRS485G-S08-R, mylib:SOP-8, symbol Interface_UART:MAX3485
- added U4: MCP2562-E-P, Package_DIP:DIP-8_W7.62mm, symbol Interface_CAN_LIN:MCP2562-E-P
- added U5: BA05CC0FP, Package_TO_SOT_SMD:TO-252-2, symbol bp5293-50:L7805
- added U7: STM32G431KBTx, Package_QFP:LQFP-32_7x7mm_P0.8mm, symbol MCU_ST_STM32G4:STM32G431KBTx
- C1, C16, C17: footprint (none) -> Capacitor_SMD:C_0603_1608Metric_Pad1.08x0.95mm_HandSolder
- C13: footprint Capacitor_THT:CP_Radial_D5.0mm_P2.00mm -> Capacitor_THT:CP_Radial_D6.3mm_P2.50mm
- C8: value 16V 100u -> 16V 220u; footprint Capacitor_THT:CP_Radial_D5.0mm_P2.00mm -> Capacitor_THT:CP_Radial_D6.3mm_P2.50mm
- D1, D2, D3: footprint MyLib:SOD123 -> mylib:SOD123
- D6, D9: footprint (none) -> LED_THT:LED_D3.0mm
- J2: footprint (none) -> Connector_JST:JST_XH_B2B-XH-A_1x02_P2.50mm_Vertical
- J3: value Conn_01x05_Socket_Encoder1 -> Conn_01x05_Socket_Encoder4; footprint (none) -> mylib:Pocket_Header_ver
- J4: footprint (none) -> mylib:Pocket_Header_ver
- J5: value Conn_01x05_Socket_Encoder1 -> Conn_01x05_Socket_Encoder2; footprint (none) -> mylib:Pocket_Header_ver
- J6: value Conn_01x05_Socket_Encoder1 -> Conn_01x05_Socket_Encoder5; footprint (none) -> mylib:Pocket_Header_ver
- J8: value Conn_01x05_Socket_Encoder1 -> Conn_01x05_Socket_Encoder3; footprint (none) -> mylib:Pocket_Header_ver
- R10, R11, R13, R14, R15, R16, R17, R18, R20, R22, R23, R9: footprint (none) -> Resistor_SMD:R_0603_1608Metric_Pad0.98x0.95mm_HandSolder
- R12: value 10k -> 4.7k; footprint (none) -> Resistor_SMD:R_0603_1608Metric_Pad0.98x0.95mm_HandSolder
- R19: value 4.7k -> 1k; footprint (none) -> Resistor_SMD:R_0603_1608Metric_Pad0.98x0.95mm_HandSolder
- R21: value 1k -> 4.7k; footprint (none) -> Resistor_SMD:R_0603_1608Metric_Pad0.98x0.95mm_HandSolder
- R25: renamed from R24; footprint (none) -> Resistor_SMD:R_0603_1608Metric_Pad0.98x0.95mm_HandSolder
- R8: value 4.7k -> 10k; footprint (none) -> Resistor_SMD:R_0603_1608Metric_Pad0.98x0.95mm_HandSolder
- SW1, SW2, SW4: footprint (none) -> Button_Switch_THT:SW_PUSH_6mm_H4.3mm
- SW3: footprint (none) -> mylib:DIP_sw_02_9.7_6.7
- U3: footprint Package_SO:SOP-8_3.9x4.9mm_P1.27mm -> mylib:SOP-8
- U6: value BP5293-50 -> BA033CC0FP; footprint MyLib:BP5293-50 -> Package_TO_SOT_SMD:TO-252-2
Connections:
- net +12V: now also R8.1; no longer R12.1
- net +3V3: now also C12.1, C13.1, C16.1, R14.1, R22.1, R23.1, R25.1, U6.3 (OUT), D5.2 (A), D8.1 (K), J7.1 (Pin_1), R24.1, U4.5 (Vio), U7.1 (VDD), U7.15 (VDDA), U7.17 (VDD)
- net +5V: now also C17.1, R10.1, R11.1, R12.1, R15.1, R16.1, R17.1, R18.1, R20.1, R21.1, R9.1, U6.1 (IN), D5.1 (K), J7.8 (Pin_8), U2.2 (~{RE}), U2.3 (DE), U2.8 (VCC), U4.3 (VDD), U5.3 (OUT); no longer U3.2 (~{RE}), U3.3 (DE), U6.3 (OUT)
- net CAN_RD: now also U4.4 (RXD), U7.21 (PA11)
- net CAN_TD: now also U4.1 (TXD), U7.22 (PA12)
- net CAN_num1: now also R23.2, U7.12 (PA7); no longer R22.2
- net CAN_num2: now also R24.2, U7.13 (PB0); no longer R23.2
- net En1_A: now also R10.2, U7.18 (PA8); no longer R9.1
- net En1_B: now also R12.2, U7.19 (PA9); no longer R11.1
- net En2_A: now also R15.2, U7.5 (PA0); no longer R15.1
- net En2_B: now also R17.2, U7.6 (PA1); no longer R17.1
- net En3_A: now also R20.2, U7.11 (PA6); no longer R19.1
- net En3_B: now also R21.2, U7.9 (PA4); no longer R20.1
- net En4_A: now also R9.2, U7.29 (PB6); no longer R8.1
- net En4_B: now also R11.2, U7.30 (PB7); no longer R10.1
- net En5_A: now also R16.2, U7.25 (PA15); no longer R16.1
- net En5_B: now also R18.2, SW1.1, U7.31 (PB8); no longer R18.1, SW1.2
- net GND: now also C17.2, SW1.2, SW2.2, U3.2 (~{RE}), U3.3 (DE), D4.1 (K), D7.1 (K), D8.2 (A), J1.1 (Pin_1), J7.12 (Pin_12), J7.5 (Pin_5), U2.5 (GND), U4.2 (VSS), U4.8 (STBY), U5.2 (GND), U7.14 (VSSA), U7.16 (VSS), U7.32 (VSS); no longer C17.1, R10.2, R11.2, R15.2, R16.2, R17.2, R18.2, R19.2, R20.2, R8.2, R9.2, SW2.1
- net RS485_RX: now also U3.1 (RO), J7.6 (Pin_6), U7.8 (PA3)
- net RS485_TX: now also J7.4 (Pin_4), U2.4 (DI), U7.7 (PA2)
- net User_LED: now also R19.1, U7.10 (PA5); no longer R21.1
- net User_button: now also U7.28 (PB5)
- net at R14.2: now also D7.2 (A)
- net at J2.1 (Pin_1), R7.1: now also U4.7 (CANH)
- net at J2.2 (Pin_2), R7.2: now also U4.6 (CANL)
- net at R2.1, R4.2: now also J1.2 (Pin_2), U2.6 (A); no longer U3.6 (A)
- net at D9.2 (A): now also R19.2; no longer R21.2
- net at R2.2, R3.1: now also J1.3 (Pin_3), U2.7 (B); no longer U3.7 (B)
- net at R1.1, R6.2: now also U3.6 (A), J1.4 (Pin_4)
- net at C5.1, C6.1, D1.1 (K)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: now also U5.1 (IN); no longer U6.1 (IN)
- net at R1.2, R5.1: now also U3.7 (B), J1.5 (Pin_5)
- removed net +3.3V: C12.1, C13.1, C16.1, R14.1, R22.1, R23.1, R25.1, SW1.1
- new net: D4.2 (A), R8.2
- new net MCO_IN: J7.10 (Pin_10), U7.2 (PF0)
- new net RESET: J7.9 (Pin_9), R22.2, SW2.1, U7.4 (PG10)
- new net SWCLK: J7.3 (Pin_3), U7.24 (PA14)
- new net SWDIO: J7.7 (Pin_7), U7.23 (PA13)
- no-connect marks 19 -> 13
Other:
- note added: "3V3に統一しましょう 済"
- note added: "5ピンのコネクタに変更して GNDを追加してください GNDは1ピンとしてください 済"
- note added: "Bootを3V3接続から GND接続に変更しました"
- note added: "FDCAN"
- note added: "RX"
- note added: "STのチップマイコンを使用する場合は ST-Linkコネクタを載せましょう ここにピンソケットをつけて線でST-Linkのボードにつなぐ 済"
- note added: "TX"
- note added: "VDDは全てに接続しましょう"
- note added: "VSSも全てに接続しましょう"
- note added: "エンコーダのA相B相はプルアップしてください 抵抗値、電源電圧は合っています 済"
- note added: "発熱敵にBA05CC0FPで耐えることが 判明したので変更しましょう 済"
- note removed: "CAN"
- moved on the sheet: R25

Commit message: 部品を配置
Parts:
- added C18: 0.1u, Capacitor_SMD:C_0603_1608Metric_Pad1.08x0.95mm_HandSolder, symbol Device:C
Connections:
- net +3V3: now also C18.1; no longer R22.1
- net +5V: now also R22.1
- net CAN_num2: now also U7.10 (PA5); no longer U7.13 (PB0)
- net GND: now also C18.2
- net User_LED: now also U7.13 (PB0); no longer U7.10 (PA5)
Changed lines of the file:
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@@
 	(wire
 		(pts
+			(xy 228.6 38.1) (xy 228.6 40.64)
+		)
+		(stroke
+			(width 0)
+			(type default)
+		)
+	)
+	(wire
+		(pts
 			(xy 236.22 78.74) (xy 236.22 81.28)
 		)
@@
 	(wire
 		(pts
+			(xy 228.6 48.26) (xy 228.6 50.8)
+		)
+		(stroke
+			(width 0)
+			(type default)
+		)
+	)
+	(wire
+		(pts
 			(xy 100.33 165.1) (xy 100.33 184.15)
 		)
@@
 	(global_label "User_LED"
 		(shape input)
-		(at 294.64 63.5 0)
+		(at 264.16 63.5 180)
 		(fields_autoplaced yes)
 		(effects
@@
 				(size 1.27 1.27)
 			)
-			(justify left)
+			(justify right)
 		)
 		(property "Intersheetrefs" "${INTERSHEET_REFS}"
-			(at 306.2733 63.5 0)
+			(at 252.5267 63.5 0)
 			(effects
 				(font
 					(size 1.27 1.27)
 				)
-				(justify left)
+				(justify right)
 				(hide yes)
 			)
@@
 	(global_label "CAN_num2"
 		(shape input)
-		(at 264.16 63.5 180)
+		(at 294.64 63.5 0)
 		(fields_autoplaced yes)
 		(effects
@@
 				(size 1.27 1.27)
 			)
-			(justify right)
+			(justify left)
 		)
 		(property "Intersheetrefs" "${INTERSHEET_REFS}"
-			(at 251.3173 63.5 0)
+			(at 307.4827 63.5 0)
 			(effects
 				(font
 					(size 1.27 1.27)
 				)
-				(justify right)
+				(justify left)
 				(hide yes)
 			)
@@
 	)
 	(symbol
+		(lib_name "GND_4")
+		(lib_id "power:GND")
+		(at 228.6 50.8 0)
+		(unit 1)
+		(exclude_from_sim no)
+		(in_bom yes)
+		(on_board yes)
+		(dnp no)
+		(property "Reference" "#PWR077"
+			(at 228.6 57.15 0)
+			(effects
+				(font
+					(size 1.27 1.27)
+				)
+				(hide yes)
+			)
+		)
+		(property "Value" "GND"
+			(at 228.6 54.61 0)
+			(effects
+				(font
+					(size 1.27 1.27)
+				)
+			)
+		)
+		(property "Footprint" ""
+			(at 228.6 50.8 0)
+			(effects
+				(font
+					(size 1.27 1.27)
+				)
+				(hide yes)
+			)
+		)
+		(property "Datasheet" ""
+			(at 228.6 50.8 0)
+			(effects
+				(font
+					(size 1.27 1.27)
+				)
+				(hide yes)
+			)
+		)
+		(property "Description" "Power symbol creates a global label with name \"GND\" , ground"
+			(at 228.6 50.8 0)
+			(effects
+				(font
+					(size 1.27 1.27)
+				)
+				(hide yes)
+			)
+		)
+		(pin "1"
+		)
+		(instances
+			(project "Encoder_board"
+				(path "/96c33453-f1dd-492b-8355-2f1b0e5bceff"
+					(reference "#PWR077")
+					(unit 1)
+				)
+			)
+		)
+	)
+	(symbol
 		(lib_name "GND_9")
 		(lib_id "power:GND")
@@
 			)
 		)
-		(property "Value" "+3V3"
+		(property "Value" "+5V"
 			(at 375.92 67.31 0)
 			(effects
@@
 	)
 	(symbol
+		(lib_id "Device:C")
+		(at 228.6 44.45 0)
+		(unit 1)
+		(exclude_from_sim no)
+		(in_bom yes)
+		(on_board yes)
+		(dnp no)
+		(fields_autoplaced yes)
+		(property "Reference" "C18"
+			(at 232.41 43.1799 0)
+			(effects
+				(font
+					(size 1.27 1.27)
+				)
+				(justify left)
+			)
+		)
+		(property "Value" "0.1u"
+			(at 232.41 45.7199 0)
+			(effects
+				(font
+					(size 1.27 1.27)
+				)
+				(justify left)
+			)
+		)
+		(property "Footprint" "Capacitor_SMD:C_0603_1608Metric_Pad1.08x0.95mm_HandSolder"
+			(at 229.5652 48.26 0)
+			(effects
+				(font
+					(size 1.27 1.27)
+				)
+				(hide yes)
+			)
+		)
+		(property "Datasheet" "~"
+			(at 228.6 44.45 0)
+			(effects
+				(font
+					(size 1.27 1.27)
+				)
+				(hide yes)
+			)
+		)
+		(property "Description" "Unpolarized capacitor"
+			(at 228.6 44.45 0)
+			(effects
+				(font
+					(size 1.27 1.27)
+				)
+				(hide yes)
+			)
+		)
+		(pin "1"
+		)
+		(pin "2"
+		)
+		(instances
+			(project "Encoder_board"
+				(path "/96c33453-f1dd-492b-8355-2f1b0e5bceff"
+					(reference "C18")
+					(unit 1)
+				)
+			)
+		)
+	)
+	(symbol
 		(lib_id "power:+3V3")
 		(at 26.67 254 0)
@@
 					(unit 1)
 				)
+			)
+		)
+	)
+	(symbol
+		(lib_name "+3V3_2")
+		(lib_id "power:+3V3")
+		(at 228.6 38.1 0)
+		(unit 1)
+		(exclude_from_sim no)
+		(in_bom yes)
+		(on_board yes)
+		(dnp no)
+		(fields_autoplaced yes)
+		(property "Reference" "#PWR076"
+			(at 228.6 41.91 0)
+			(effects
+				(font
+					(size 1.27 1.27)
+				)
+				(hide yes)
+			)
+		)
+		(property "Value" "+3V3"
+			(at 228.6 33.02 0)
+			(effects
+				(font
+					(size 1.27 1.27)
+				)
+			)
+		)
+		(property "Footprint" ""
+			(at 228.6 38.1 0)
+			(effects
+				(font
+					(size 1.27 1.27)
+				)
+				(hide yes)
+			)
+		)
+		(property "Datasheet" ""
+			(at 228.6 38.1 0)
+			(effects
+				(font
+					(size 1.27 1.27)
+				)
+				(hide yes)
+			)
+		)
+		(property "Description" "Power symbol creates a global label with name \"+3V3\""
+			(at 228.6 38.1 0)
+			(effects
+				(font
+					(size 1.27 1.27)
+				)
+				(hide yes)
+			)
+		)
+		(pin "1"
+		)
+		(instances
+			(project "Encoder_board"
+				(path "/96c33453-f1dd-492b-8355-2f1b0e5bceff"
+					(reference "#PWR076")
+					(unit 1)
+				)

Commit message: 配線終了。あとはシルク
Parts:
- SW3: footprint mylib:DIP_sw_02_9.7_6.7 -> Button_Switch_THT:SW_DIP_SPSTx02_Slide_6.7x6.64mm_W7.62mm_P2.54mm_LowProfile
Connections:
- net +3V3: now also R22.1
- net +5V: no longer R22.1
Changed lines of the file:
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@@
 			)
 		)
-		(property "Footprint" "mylib:DIP_sw_02_9.7_6.7"
+		(property "Footprint" "Button_Switch_THT:SW_DIP_SPSTx02_Slide_6.7x6.64mm_W7.62mm_P2.54mm_LowProfile"
 			(at 397.51 49.53 0)
 			(effects
@@
 		(on_board yes)
 		(dnp no)
-		(fields_autoplaced yes)
 		(property "Reference" "#PWR070"
 			(at 375.92 76.2 0)
@@
 			)
 		)
-		(property "Value" "+5V"
-			(at 375.92 67.31 0)
-			(effects
-				(font
-					(size 1.27 1.27)
-				)
-			)
-		)
+		(property "Value" "+3V3"
+			(at 373.38 68.58 0)
+			(effects
+				(font
+					(size 1.27 1.27)
+				)
+				(justify left)
+			)
+		)
