File: Encoder_board.kicad_pcb (KiCad board)
At the start: 2 copper layers, 70 x 70 mm, 77 parts, among them J1 Conn_01x05_Socket_RS485, J2 CAN_OUT, J3 Conn_01x05_Socket_Encoder4, J4 Conn_01x05_Socket_Encoder1, J5 Conn_01x05_Socket_Encoder2, J6 Conn_01x05_Socket_Encoder5, J7 ST-Link_pinsocket, J8 Conn_01x05_Socket_Encoder3, SW1 SW_Boot, SW2 SW_Reset, SW3 SW_DIP_x02_CANnum, SW4 SW_User, U1 XT60_M, U2 UTRS485G-S08-R, U3 UTRS485G-S08-R, U4 MCP2562-E-P, U5 BA05CC0FP, U6 BA033CC0FP, U7 STM32G431KBTx

Commit message: コメントをPCBエディタに追加
Other:
- board text added: "En_1のエンコーダへの5Vが細いかも いや太さ的には足りるんですけど、ここだけ他と違う太さなの気になります。"
- board text added: "ST＿Linkのシルクなんですけど ーーーーーーーーーーーーーーー→ TXRX以外も書いていただけると挿し違いが減って嬉しいです"
- board text added: "TXとRXの部分、AかBかも書いておくと見やすいです(回路図参照）ーーーーーーーーー→ あとGNDも。"
- board text added: "UserButtonとUserLEDも、隣にPB5とかPB0とか書いてあると制御に優しいです"
- board text added: "←CAN_numからboard_num に変更していたただいても良いですかね 通信にはRS-485も使えるのでCANに縛らない方が良いかなって"
- board text added: "←Cxxなどの各リファレンス番号は同じ向きに揃えておくとはんだ付けの際に見やすいのでおすすめです。"
- board text added: "ビアいっぱいあって良いですね。 一応こんなに打たなくても十分らしいです。３−5mmに一個くらい。でも足りないより多いほうが良いのでOK 基板の空いてるところをビアで埋めるのがめんどくさい場合は、ビア打ておじさんを使うと楽です。 こちら→https://github.com/KeioRoboticsAssociation/Via_Ute_Ojisan"
- board text added: "全体的に配線がスッキリしていて良いすね 直角に交わるところもないように工夫したり、電流多い配線はビア多めに打ったりしててナイスです"
- board text added: "各エンコーダコネクタにEn_xと書いてて良いですね ついでにそれらがどのタイマーなのか、Tim1とかTim2とか 書いてあると制御に優しいです。"
- board text added: "基板設定ー＞デザインルールー＞制約ー＞導体から基板端クリアランス は０にして大丈夫です 基板の端っこも塗りつぶされるようになります。"
- board text added: "裏にB.Silkscreenで大きめの塗りつぶし矩形を置いておくと、 マッキーとかで記入できるスペースを設けられるのでおすすめです。 これくらいの→"
Changed lines of the file:
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@@
 		)
 		(property "Value" "Conn_01x05_Socket_Encoder1"
-			(at 0 14.5 180)
+			(at -0.04 2.8 180)
 			(unlocked yes)
 			(layer "F.Fab")
@@
 		(layer "B.Cu")
 	)
+	(gr_rect
+		(start 146.685 162.179)
+		(end 172.339 165.862)
+		(stroke
+			(width 0.1)
+			(type solid)
+		)
+		(fill yes)
+		(layer "B.SilkS")
+	)
 	(gr_line
 		(start 178.503998 62.5)
@@
 			)
 			(justify left bottom)
+		)
+	)
+	(gr_text "各エンコーダコネクタにEn_xと書いてて良いですね\nついでにそれらがどのタイマーなのか、Tim1とかTim2とか\n書いてあると制御に優しいです。"
+		(at 110.49 137.541 0)
+		(layer "User.2")
+		(effects
+			(font
+				(size 1 1)
+				(thickness 0.15)
+			)
+			(justify left bottom)
+		)
+	)
+	(gr_text "TXとRXの部分、AかBかも書いておくと見やすいです(回路図参照）ーーーーーーーーー→\nあとGNDも。"
+		(at 71.12 121.793 0)
+		(layer "User.2")
+		(effects
+			(font
+				(size 1 1)
+				(thickness 0.15)
+			)
+			(justify left bottom)
+		)
+	)
+	(gr_text "基板設定ー＞デザインルールー＞制約ー＞導体から基板端クリアランス\nは０にして大丈夫です\n基板の端っこも塗りつぶされるようになります。"
+		(at 84.709 45.339 0)
+		(layer "User.2")
+		(effects
+			(font
+				(size 1 1)
+				(thickness 0.1)
+			)
+			(justify left bottom)
+		)
+	)
+	(gr_text "←Cxxなどの各リファレンス番号は同じ向きに揃えておくとはんだ付けの際に見やすいのでおすすめです。"
+		(at 173.355 84.455 0)
+		(layer "User.2")
+		(effects
+			(font
+				(size 1 1)
+				(thickness 0.15)
+			)
+			(justify left bottom)
+		)
+	)
+	(gr_text "←CAN_numからboard_num\nに変更していたただいても良いですかね\n通信にはRS-485も使えるのでCANに縛らない方が良いかなって"
+		(at 175.768 113.538 0)
+		(layer "User.2")
+		(effects
+			(font
+				(size 1 1)
+				(thickness 0.15)
+			)
+			(justify left bottom)
+		)
+	)
+	(gr_text "ビアいっぱいあって良いですね。\n一応こんなに打たなくても十分らしいです。３−5mmに一個くらい。でも足りないより多いほうが良いのでOK\n基板の空いてるところをビアで埋めるのがめんどくさい場合は、ビア打ておじさんを使うと楽です。\nこちら→https://github.com/KeioRoboticsAssociation/Via_Ute_Ojisan"
+		(at 110.871 155.829 0)
+		(layer "User.2")
+		(effects
+			(font
+				(size 1 1)
+				(thickness 0.15)
+			)
+			(justify left bottom)
+		)
+	)
+	(gr_text "ST＿Linkのシルクなんですけど ーーーーーーーーーーーーーーー→\nTXRX以外も書いていただけると挿し違いが減って嬉しいです"
+		(at 87.122 100.076 0)
+		(layer "User.2")
+		(effects
+			(font
+				(size 1 1)
+				(thickness 0.1)
+			)
+			(justify left bottom)
+		)
+	)
+	(gr_text "裏にB.Silkscreenで大きめの塗りつぶし矩形を置いておくと、\nマッキーとかで記入できるスペースを設けられるのでおすすめです。\nこれくらいの→"
+		(at 110.998 166.624 0)
+		(layer "User.2")
+		(effects
+			(font
+				(size 1 1)
+				(thickness 0.15)
+			)
+			(justify left bottom)
+		)
+	)
+	(gr_text "En_1のエンコーダへの5Vが細いかも\nいや太さ的には足りるんですけど、ここだけ他と違う太さなの気になります。"
+		(at 131.572 56.134 0)
+		(layer "User.2")
+		(effects
+			(font
+				(size 1 1)
+				(thickness 0.15)
+			)
+			(justify left bottom)
+		)
+	)
+	(gr_text "UserButtonとUserLEDも、隣にPB5とかPB0とか書いてあると制御に優しいです"
+		(at 110.744 143.891 0)
+		(layer "User.2")
+		(effects
+			(font
+				(size 1 1)
+				(thickness 0.15)
+			)
+			(justify left bottom)
+		)
+	)
+	(gr_text "全体的に配線がスッキリしていて良いすね\n直角に交わるところもないように工夫したり、電流多い配線はビア多めに打ったりしててナイスです"
+		(at 197.358 143.256 0)
+		(layer "User.2")
+		(effects
+			(font
+				(size 1 1)
+				(thickness 0.1)
+			)
+			(justify left bottom)

Commit message: コメントをPCBエディタに追加
Other:
- board text added: "どこかにF.Silkscreenで JLCJLCJLCJLC と記述しておくと、そこに基板の製造番号位置を指定できます。おすすめです。"
Changed lines of the file:
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@@
+		)
+	)
+	(gr_text "どこかにF.Silkscreenで\nJLCJLCJLCJLC\nと記述しておくと、そこに基板の製造番号位置を指定できます。おすすめです。"
+		(at 110.998 174.498 0)
+		(layer "User.2")
+		(effects
+			(font
+				(size 1 1)
+				(thickness 0.15)
+			)
+			(justify left bottom)
 		)
 	)
