File: Encoder_board.kicad_pcb (KiCad board)
At the start: 2 copper layers, 70 x 70 mm, 77 parts, among them J1 Conn_01x05_Socket_RS485, J2 CAN_OUT, J3 Conn_01x05_Socket_Encoder4, J4 Conn_01x05_Socket_Encoder1, J5 Conn_01x05_Socket_Encoder2, J6 Conn_01x05_Socket_Encoder5, J7 ST-Link_pinsocket, J8 Conn_01x05_Socket_Encoder3, SW1 SW_Boot, SW2 SW_Reset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

Commit message: 修正完了
Connections:
- net CAN_num1 renamed board_num1
- net CAN_num2 renamed board_num2
- net En1_A renamed En1_A_Tim1_CH1
- net En1_B renamed En1_B_Tim1_CH2
- net En2_A renamed En2_A_Tim2_CH1
- net En2_B renamed En2_B_Tim2_CH2
- net En3_A renamed En3_A_Tim3_CH1
- net En3_B renamed En3_B_Tim3_CH2
- net En4_A renamed En4_A_Tim4_CH1
- net En4_B renamed En4_B_Tim4_CH2
- net En5_A renamed En5_A_Tim8_CH1
- net En5_B renamed En5_B_Tim8_CH2
Routing:
- net GND: vias 1435 -> 1429
Other:
- board text added: "CLK"
- board text added: "DIO"
- board text added: "En_1_Tim1"
- board text added: "En_2_Tim2"
- board text added: "En_3_Tim3"
- board text added: "En_4_Tim4"
- board text added: "En_5_Iim8"
- board text added: "JLCJLCJLCJLC"
- board text added: "MCO"
- board text added: "PA5"
- board text added: "PA7"
- board text added: "RST"
- board text added: "RXA"
- board text added: "RXB"
- board text added: "TXA"
- board text added: "TXB"
- board text added: "User_LED_PB0"
- board text added: "User_PB5"
- board text added: "board_num"
- board text removed: "CAN_num"
- board text removed: "En_1"
- board text removed: "En_2"
- board text removed: "En_3"
- board text removed: "En_4"
- board text removed: "En_5"
- board text removed: "User"
- board text removed: "User_LED"
